Commit message: added end effector to robot

File: src/robot_description/urdf/robot_macro.xacro (robot description, xacro)
@@ -85,4 +85,18 @@
       <origin xyz="0 0 0" rpy="0 0 0" />
     </xacro:ur_robot>
-  </xacro:macro>
+    <!-- End effector link -->
+    <link name="end_effector_link">
+        <visual>
+            <geometry>
+                <mesh filename="package://robot_description/meshes/Gripper_fixed.stl" scale="0.001 0.001 0.001"/>
+            </geometry>
+            <origin xyz="-0.124 0 0.04" rpy="0 3.1416 0"/>
+        </visual>
+    </link>
+    <!-- Coupler between arm and end effector -->
+    <joint name="end_effector_coupler_joint" type="fixed">
+        <parent link="${ur_type}_tool0"/>
+        <child link="end_effector_link"/>
+    </joint>
+    </xacro:macro>
 </robot>

Commit message: finished setup assistant

File: src/robot_description/urdf/robot_macro.xacro (robot description, xacro)
@@ -93,4 +93,9 @@
             <origin xyz="-0.124 0 0.04" rpy="0 3.1416 0"/>
         </visual>
+        <collision>
+            <geometry>
+                <box size="0.248 0.30 0.30"/>
+            </geometry>
+        </collision>
     </link>
     <!-- Coupler between arm and end effector -->

Commit message: fixing setup assistant issues

File: src/robot_description/urdf/robot_macro.xacro (robot description, xacro)
@@ -95,6 +95,7 @@
         <collision>
             <geometry>
-                <box size="0.248 0.30 0.30"/>
+                <box size="0.2 0.075 0.20"/>
             </geometry>
+            <origin xyz="0 0 0.1" rpy="0 3.1416 0"/>
         </collision>
     </link>
