Commit message: Implemented robot_description

File: src/robot_description/urdf/burger_bot.xacro (robot description, xacro)
@@ -5,4 +5,9 @@
   <xacro:include filename="$(find ur_description)/urdf/ur.urdf.xacro"/>
   <!---Table-->
+  <xacro:include filename="table.urdf"/>
+  <joint name="table_link_joint" type="fixed">
+    <parent link="base_link"/>
+    <child link="table_link"/>
+  </joint>
   <!--End Effector-->
   <xacro:include filename="end_effector.urdf"/>

File: src/robot_description/urdf/end_effector.urdf (robot description, URDF)
Before this commit: robot end_effector.urdf, 1 links, 0 joints
Links:
- link end_effector_link: geometry collision box size=0.342 0.087 0.130; visual mesh filename=package://robot_description/meshes/EndEffector.obj
