Commit message: real testing

File: src/robot_description/urdf/end_effector.urdf (robot description, URDF)
Before this commit: robot end_effector.urdf, 1 links, 0 joints
Links:
- link end_effector_link: geometry collision box size=0.30 0.087 0.130; collision box size=0.342 0.087 0.130

Commit message: fixed rotation issue and adjusted end effector collision box

File: src/robot_description/urdf/end_effector.urdf (robot description, URDF)
Before this commit: robot end_effector.urdf, 1 links, 0 joints
Links:
- link end_effector_link: geometry collision box size=0.268 0.087 0.097; collision box size=0.342 0.087 0.033
