Commit message: conforming to humble format of setup assistant

File: src/burger_bot_cell/burger_bot_description/urdf/burger_bot.urdf.xacro (robot description, xacro)
@@ -1,5 +1,5 @@
 <?xml version="1.0"?>
-<robot name="robot" xmlns:xacro="http://ros.org/wiki/xacro">
-  <xacro:include filename="$(find robot_description)/urdf/robot_macro.xacro"/>
+<robot name="burger_bot_cell" xmlns:xacro="http://ros.org/wiki/xacro">
+  <xacro:include filename="$(find burger_bot_description)/urdf/burger_bot_macro.xacro"/>
   <xacro:arg name="ur_type" default="ur5e"/>
   <xacro:arg name="joint_limits_parameters_file" default="$(find ur_description)/config/$(arg ur_type)/joint_limits.yaml"/>
@@ -9,5 +9,5 @@
   <link name="world"/>
   <!--This will create the scene where the robot is located in-->
-  <xacro:robot_cell
+  <xacro:burger_bot_cell
     parent="world"
     ur_type="$(arg ur_type)"
@@ -17,5 +17,5 @@
     visual_parameters_file="$(arg visual_parameters_file)"
     >
-      <origin xyz="0 0 0" rpy="0 0 0" />
-  </xacro:robot_cell>
+      <origin xyz="0 0 1" rpy="0 0 0" />
+  </xacro:burger_bot_cell>
 </robot>

File: src/burger_bot_cell/burger_bot_description/urdf/burger_bot_macro.xacro (robot description, xacro)
@@ -2,5 +2,5 @@
 <robot xmlns:xacro="http://ros.org/wiki/xacro">
   <xacro:include filename="$(find ur_description)/urdf/ur_macro.xacro"/>
-  <xacro:macro name="robot_cell" params="
+  <xacro:macro name="burger_bot_cell" params="
     parent
     *origin
@@ -19,5 +19,5 @@
       <visual>
         <geometry>
-          <mesh filename="package://robot_description/meshes/fzi_table.dae"/>
+          <mesh filename="package://burger_bot_description/meshes/fzi_table.dae"/>
         </geometry>
         <origin rpy="0 0 0" xyz="0.75 0.5 -1"/>
@@ -25,5 +25,5 @@
       <collision>
         <geometry>
-          <mesh filename="package://robot_description/meshes/fzi_table.dae"/>
+          <mesh filename="package://burger_bot_description/meshes/fzi_table.dae"/>
         </geometry>
         <origin rpy="0 0 0" xyz="0.75 0.5 -1"/>
@@ -33,10 +33,10 @@
       <visual>
         <geometry>
-          <mesh filename="package://robot_description/meshes/171005_Motek_Monitor_L.dae"/>
+          <mesh filename="package://burger_bot_description/meshes/171005_Motek_Monitor_L.dae"/>
         </geometry>
       </visual>
       <collision>
         <geometry>
-          <mesh filename="package://robot_description/meshes/171005_Motek_Monitor_L.dae"/>
+          <mesh filename="package://burger_bot_description/meshes/171005_Motek_Monitor_L.dae"/>
         </geometry>
       </collision>
@@ -53,5 +53,5 @@
       <visual>
         <geometry>
-          <mesh filename="package://robot_description/meshes/wall.dae"/>
+          <mesh filename="package://burger_bot_description/meshes/wall.dae"/>
         </geometry>
       </visual>
@@ -82,4 +82,5 @@
       physical_parameters_file="${physical_parameters_file}"
       visual_parameters_file="${visual_parameters_file}"
+      generate_ros2_control_tag="false"
     >
       <origin xyz="0 0 0" rpy="0 0 0" />
@@ -89,5 +90,5 @@
         <visual>
             <geometry>
-                <mesh filename="package://robot_description/meshes/Gripper_fixed.stl" scale="0.001 0.001 0.001"/>
+                <mesh filename="package://burger_bot_description/meshes/Gripper_fixed.stl" scale="0.001 0.001 0.001"/>
             </geometry>
             <origin xyz="-0.124 0 0.04" rpy="0 3.1416 0"/>
@@ -105,4 +106,4 @@
         <child link="end_effector_link"/>
     </joint>
-    </xacro:macro>
+  </xacro:macro>
 </robot>

Commit message: successfully completed controll module

File: src/burger_bot_cell/burger_bot_description/urdf/burger_bot.urdf.xacro (robot description, xacro)
@@ -2,5 +2,5 @@
 <robot name="burger_bot_cell" xmlns:xacro="http://ros.org/wiki/xacro">
   <xacro:include filename="$(find burger_bot_description)/urdf/burger_bot_macro.xacro"/>
-  <xacro:arg name="ur_type" default="ur5e"/>
+  <xacro:arg name="ur_type" default="ur20"/>
   <xacro:arg name="joint_limits_parameters_file" default="$(find ur_description)/config/$(arg ur_type)/joint_limits.yaml"/>
   <xacro:arg name="kinematics_parameters_file" default="$(find ur_description)/config/$(arg ur_type)/default_kinematics.yaml"/>

File: src/burger_bot_cell/burger_bot_description/urdf/burger_bot_macro.xacro (robot description, xacro)
@@ -86,24 +86,4 @@
       <origin xyz="0 0 0" rpy="0 0 0" />
     </xacro:ur_robot>
-    <!-- End effector link -->
-    <link name="end_effector_link">
-        <visual>
-            <geometry>
-                <mesh filename="package://burger_bot_description/meshes/Gripper_fixed.stl" scale="0.001 0.001 0.001"/>
-            </geometry>
-            <origin xyz="-0.124 0 0.04" rpy="0 3.1416 0"/>
-        </visual>
-        <collision>
-            <geometry>
-                <box size="0.2 0.075 0.20"/>
-            </geometry>
-            <origin xyz="0 0 0.1" rpy="0 3.1416 0"/>
-        </collision>
-    </link>
-    <!-- Coupler between arm and end effector -->
-    <joint name="end_effector_coupler_joint" type="fixed">
-        <parent link="${ur_type}_tool0"/>
-        <child link="end_effector_link"/>
-    </joint>
   </xacro:macro>
 </robot>

Commit message: successfully controlling with the inbuilt moveit gui

File: src/burger_bot_cell/burger_bot_description/urdf/burger_bot.urdf.xacro (robot description, xacro)
@@ -2,5 +2,5 @@
 <robot name="burger_bot_cell" xmlns:xacro="http://ros.org/wiki/xacro">
   <xacro:include filename="$(find burger_bot_description)/urdf/burger_bot_macro.xacro"/>
-  <xacro:arg name="ur_type" default="ur20"/>
+  <xacro:arg name="ur_type" default="ur5e"/>
   <xacro:arg name="joint_limits_parameters_file" default="$(find ur_description)/config/$(arg ur_type)/joint_limits.yaml"/>
   <xacro:arg name="kinematics_parameters_file" default="$(find ur_description)/config/$(arg ur_type)/default_kinematics.yaml"/>

File: src/burger_bot_cell/burger_bot_description/urdf/burger_bot_macro.xacro (robot description, xacro)
@@ -86,4 +86,22 @@
       <origin xyz="0 0 0" rpy="0 0 0" />
     </xacro:ur_robot>
+    <link name="end_effector_link">
+      <visual>
+        <geometry>
+          <mesh filename="package://burger_bot_description/meshes/Gripper_fixed.stl" scale="0.001 0.001 0.001"/>
+        </geometry>
+        <origin xyz="-0.124 0 0.04" rpy="0 3.1416 0"/>
+      </visual>
+      <collision>
+        <geometry>
+          <box size="0.2, 0.075, 0.2"/>
+        </geometry>
+        <origin xyz="-0.124 0 0.04" rpy="0 3.1416 0"/>
+      </collision>
+    </link>
+    <joint name="end_effector_link_joint" type="fixed">
+      <parent link="${ur_type}_tool0"/>
+      <child link="end_effector_link"/>
+    </joint>
   </xacro:macro>
 </robot>
