Commit message: fixing

File: src/burger_bot_cell/burger_bot_description/urdf/burger_bot_macro.xacro (robot description, xacro)
@@ -91,5 +91,5 @@
           <mesh filename="package://burger_bot_description/meshes/Gripper_fixed.stl" scale="0.001 0.001 0.001"/>
         </geometry>
-        <origin xyz="-0.124 0 0.04" rpy="0 3.1416 0"/>
+        <origin xyz="-0.124 0 0.078" rpy="0 3.1416 0"/>
       </visual>
       <collision>
@@ -97,5 +97,5 @@
           <box size="0.2, 0.075, 0.2"/>
         </geometry>
-        <origin xyz="-0.124 0 0.04" rpy="0 3.1416 0"/>
+        <origin xyz="-0.124 0 0.078" rpy="0 3.1416 0"/>
       </collision>
     </link>
@@ -106,2 +106,4 @@
   </xacro:macro>
 </robot>
+<!-- bracket link = 38mm -->
+<!-- previously 0.04 -->

Commit message: added real table to scene

File: src/burger_bot_cell/burger_bot_description/urdf/burger_bot_macro.xacro (robot description, xacro)
@@ -19,32 +19,15 @@
       <visual>
         <geometry>
-          <mesh filename="package://burger_bot_description/meshes/fzi_table.dae"/>
+          <mesh filename="package://burger_bot_description/meshes/Tablev2_v13.stl" scale="0.001 0.001 0.001"/>
         </geometry>
-        <origin rpy="0 0 0" xyz="0.75 0.5 -1"/>
+        <origin rpy="0 0 0" xyz="1 0.2 0"/>
       </visual>
       <collision>
         <geometry>
-          <mesh filename="package://burger_bot_description/meshes/fzi_table.dae"/>
+          <mesh filename="package://burger_bot_description/meshes/Tablev2_v13.stl" scale="0.001 0.001 0.001"/>
         </geometry>
-        <origin rpy="0 0 0" xyz="0.75 0.5 -1"/>
+        <origin rpy="0 0 0" xyz="0 0 0"/>
       </collision>
     </link>
-    <link name="monitor">
-      <visual>
-        <geometry>
-          <mesh filename="package://burger_bot_description/meshes/171005_Motek_Monitor_L.dae"/>
-        </geometry>
-      </visual>
-      <collision>
-        <geometry>
-          <mesh filename="package://burger_bot_description/meshes/171005_Motek_Monitor_L.dae"/>
-        </geometry>
-      </collision>
-    </link>
-    <joint name="base_to_monitor" type="fixed">
-      <parent link="table"/>
-      <child link="monitor"/>
-      <origin xyz="0.2 0.6 0"/>
-    </joint>
     <material name="white">
       <color rgba="1 1 1 1"/>
@@ -108,2 +91,3 @@
 <!-- bracket link = 38mm -->
 <!-- previously 0.04 -->
+<!-- 0.135 -0.660 0" -->
